Commit message: add cumstomized desc

File: turtlebot_description/urdf/turtlebot_gazebo.urdf.xacro (robot description, xacro)
@@ -6,5 +6,5 @@
       <sensor type="depth" name="camera">
         <always_on>true</always_on>
-        <update_rate>20.0</update_rate>
+        <update_rate>30.0</update_rate>
         <camera>
           <horizontal_fov>${60.0*M_PI/180.0}</horizontal_fov>
@@ -16,11 +16,16 @@
           <clip>
             <near>0.05</near>
-            <far>8.0</far>
+            <far>50.0</far>
           </clip>
+          <noise>
+          <type>gaussian</type>
+          <mean>0.0</mean>
+          <stddev>0.007</stddev>
+        </noise>
         </camera>
         <plugin name="kinect_camera_controller" filename="libgazebo_ros_openni_kinect.so">
           <cameraName>camera</cameraName>
           <alwaysOn>true</alwaysOn>
-          <updateRate>10</updateRate>
+          <updateRate>30</updateRate>
           <imageTopicName>rgb/image_raw</imageTopicName>
           <depthImageTopicName>depth/image_raw</depthImageTopicName>

File: turtlebot_description/urdf/turtlebot_properties_fisheye_stereo.urdf.xacro (robot description, xacro)
@@ -19,9 +19,9 @@
      (currently in development and awaiting feedback)
    -->
-  <xacro:property name="cam_px" value="0.15" />
-  <xacro:property name="cam_pz" value="0.3" />
-  <xacro:property name="cam_or" value="0" />
-  <xacro:property name="cam_op" value="0" />
-  <xacro:property name="cam_oy" value="0" />
+	<xacro:property name="cam_px" value="0.15" />
+	<xacro:property name="cam_pz" value="0.3" />
+	<xacro:property name="cam_or" value="0" />
+	<xacro:property name="cam_op" value="0" />
+	<xacro:property name="cam_oy" value="0" />
 <!--   <xacro:property name="cam_px" value="-0.087" />
   <xacro:property name="cam_pz" value="0.2870" />
